File: sdi12-analog-mux.kicad_pcb (KiCad board)
At the start: 4 copper layers, 89.5 x 49.5 mm, 117 parts, among them J1 Conn_01x02, J10 Screw_Terminal_01x04, J11 Screw_Terminal_01x04, J12 Screw_Terminal_01x04, J2 USB_B_Micro, J3 SM03B-SRSS-TB, J4 Screw_Terminal_01x03, J5 Conn_01x03_Socket, J6 Screw_Terminal_01x04, J7 Screw_Terminal_01x04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

Commit message: version 1.0 after v0.0 bringup modifications
Parts:
- removed R6: 100, Resistor_SMD:R_0402_1005Metric
- added a: LOGO, LOGO, F.Cu at (137.6, 68.6)
- added a: LOGO, LOGO, F.Cu at (110.4, 109.7)
- D2, D3, D4, D5, D6, D7, D8: footprint Diode_SMD:D_0402_1005Metric -> Diode_SMD:D_SOD-323F
- L1: footprint Capacitor_SMD:C_0402_1005Metric -> 74438334022:WE-MAPI_3012
- moved L1 1.40 mm to (101.1, 111.4)
- moved D5 1.31 mm to (169.2, 89.7), turned to 90 degrees
- moved J1 1.10 mm to (115.0, 71.3)
- moved C10 1.05 mm to (105.0, 71.5)
- moved D6 0.78 mm to (166.8, 88.3)
- moved D7 0.71 mm to (164.7, 88.3)
- moved C11 0.65 mm to (101.7, 108.3)
- moved D8 0.65 mm to (162.6, 88.3)
- moved D4 0.28 mm to (166.8, 92.9)
- moved D2 0.22 mm to (162.6, 92.9)
- moved D3 0.20 mm to (164.7, 92.9)
- turned U3 to 90 degrees
Connections:
- R29 pad 1: Net-(R19-Pad2) -> /EXCITATION_CURRENT_OUT
- R30 pad 1: GND -> Net-(R19-Pad2)
- U3 pad 3: +5V -> +3V3
- U3 pad 5: /SDI12_DATA_5V -> /SDI12_DATA_3V3
- U3 pad 6: Net-(U3-OE) -> +3V3
- U3 pad 7: +3V3 -> +5V
- U3 pad 8: /SDI12_DATA_3V3 -> /SDI12_DATA_5V
Routing:
- net +3V3: track 65.2 -> 68.5 mm, vias 36 -> 35
- net /EXCITATION_CURRENT_OUT: track 18.4 -> 21.2 mm
- net /RTD_4_NEG: track 26.9 -> 29.6 mm
- net /SDI12_DATA_5V: track 9.74 -> 7.34 mm
- net Net-(R19-Pad2): track 4.25 -> 6.20 mm
- net Net-(U3-OE): track 1.85 -> 0.00 mm
- net Net-(D5-A): track 12.9 -> 11.3 mm
- net Net-(D4-A): track 27.1 -> 25.6 mm
- net /SDI12_DATA_3V3: track 11.7 -> 10.3 mm
- net Net-(D7-A): track 19.2 -> 17.9 mm
- net Net-(D6-A): track 20.5 -> 19.2 mm
- net /RTD_4_POS: track 24.1 -> 25.2 mm
- net Net-(D8-A): track 27.3 -> 26.4 mm
- net Net-(D2-A): track 21.3 -> 20.4 mm
- net Net-(D3-A): track 19.7 -> 18.9 mm
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Other:
- outline, holes or cut-outs redrawn
- board text added: "12V"
- board text added: "DATA"
- board text added: "GND"
- board text added: "RX-ORG"
- board text added: "SDI12-Analog-Mux v1.0 Project Gorgon"
- board text added: "TX-YLW"
- board text added: "Zach Radlicz"
- board text removed: "SDI12-Analog-Mux v0.0"
